File: UniFi.kicad_pcb (KiCad board)
At the start: 2 copper layers, 120.2 x 100.1 mm, 67 parts, among them J1 OLED, J2 MJ-4PP-9 TRRS, SW1 SW_PUSH-MX_W_LED, SW10 SW_PUSH-MX_W_LED, SW11 SW_PUSH-MX_W_LED, SW12 SW_PUSH-MX_W_LED, SW13 SW_PUSH-MX_W_LED, SW14 SW_PUSH-MX_W_LED, SW15 SW_PUSH-MX_W_LED, SW16 SW_PUSH-MX_W_LED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

Commit message: Updated PCB
Connections:
- J2 pad A: A -> (no net)
- J2 pad B: B -> (no net)
- U1 pad P1: C -> (no net)
- U1 pad P10: L -> (no net)
- U1 pad P11: M -> (no net)
- U1 pad P12: N -> (no net)
- U1 pad P13: O -> (no net)
- U1 pad P14: P -> (no net)
- U1 pad P15: Q -> (no net)
- U1 pad P16: R -> (no net)
- U1 pad P17: S -> (no net)
- U1 pad P18: T -> (no net)
- U1 pad P19: U -> (no net)
- U1 pad P2: D -> (no net)
- U1 pad P20: V -> (no net)
- U1 pad P21: W -> (no net)
- U1 pad P22: X -> (no net)
- U1 pad P23: Y -> (no net)
- U1 pad P24: Z -> (no net)
- U1 pad P3: E -> (no net)
- U1 pad P4: F -> (no net)
- U1 pad P5: G -> (no net)
- U1 pad P6: H -> (no net)
- U1 pad P7: I -> (no net)
- U1 pad P8: J -> (no net)
- U1 pad P9: K -> (no net)
Routing:
- net (no net): track 0.00 -> 159.7 mm, vias 0 -> 2
- net B: track 15.8 -> 0.00 mm, vias 1 -> 0
- net A: track 15.7 -> 0.00 mm, vias 1 -> 0
- net Z: track 5.34 -> 0.00 mm
- net Y: track 5.34 -> 0.00 mm
- net X: track 5.34 -> 0.00 mm
- net W: track 5.34 -> 0.00 mm
- net V: track 5.34 -> 0.00 mm
- net U: track 5.34 -> 0.00 mm
- net T: track 5.34 -> 0.00 mm
- net S: track 5.34 -> 0.00 mm
- net R: track 5.34 -> 0.00 mm
- net Q: track 5.34 -> 0.00 mm
- net P: track 5.34 -> 0.00 mm
- net O: track 5.34 -> 0.00 mm
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