File: Plates/UniFi - Plate.kicad_pcb (KiCad board)
At the start: 2 copper layers, 120.2 x 100.1 mm, 19 parts

Commit message: Updated Plate
Other:
- outline, holes or cut-outs redrawn
- board text added: "Unifi"
